Commit message: updated inverse kinematics chain

File: Implementierung/Greifer/RescueBot_Baugruppe.SLDASM/urdf/RescueBot_Baugruppe.SLDASM.urdf (robot description, URDF)
Before this commit: robot RescueBot_Baugruppe.SLDASM, 5 links, 4 joints
Links:
- added link finger, mass 0.09972; collision mesh filename=package://RescueBot_Baugruppe.SLDASM/meshes/finger.STL; visual mesh filename=package://RescueBot_Baugruppe.SLDASM/meshes/finger.STL
- link base_link: mass 325.51 -> 3.0727
- link drehplatte: mass 0.42188 -> 3.0727
- link hand: mass 0.00679092879672445 -> 0.10222
- link oberarm: mass 0.27688 -> 2.5014
- link unterarm: mass 0.138646560275947 -> 1.0425
Joints:
- removed joint Dreplatte
- added joint Drehplatt: type fixed, parent base_link, child drehplatte, origin xyz=0 -0.8 0.44817 rpy=1.5708 0 0.10036, axis 0 0 0
- added joint Finger: type fixed, parent hand, child finger, origin xyz=0.066137 0 0.32806 rpy=3.1416 1.5708 0, axis 0 0 0
- joint Hand: origin xyz=0 0 0.430000000000003 rpy=-0.332130576060565 0 0 -> xyz=0 0 0.575 rpy=-0.82998 0 0
- joint Oberarm: axis 1 0 0 -> 0 0 1; origin xyz=0 0.06 0.015 rpy=-2.4448 0 3.1416 -> xyz=0 0.203 0.025 rpy=-1.5708 -1.2778 1.5708
- joint Unterarm: origin xyz=0 0.0150000000000005 -0.270000000000002 rpy=-2.07124984213266 0 3.14159265358979 -> xyz=0.745 0 0 rpy=1.8898 1.5708 0

Commit message: ik-chain update

File: Implementierung/Greifer/RescueBot_Baugruppe.SLDASM/urdf/RescueBot_Baugruppe.SLDASM.urdf (robot description, URDF)
Before this commit: robot RescueBot_Baugruppe.SLDASM, 6 links, 5 joints
Links:
- removed link drehplatte
- removed link finger
- removed link hand
- removed link oberarm
- removed link unterarm
- added link ellenbogen, mass 5.0028; collision mesh filename=package://RescueBot_Baugruppe.SLDASM/meshes/ellenbogen.STL; visual mesh filename=package://RescueBot_Baugruppe.SLDASM/meshes/ellenbogen.STL
- added link fingergelenk, mass 0.04986; collision mesh filename=package://RescueBot_Baugruppe.SLDASM/meshes/fingergelenk.STL; visual mesh filename=package://RescueBot_Baugruppe.SLDASM/meshes/fingergelenk.STL
- added link handgelenk, mass 2.08500049128727; collision mesh filename=package://RescueBot_Baugruppe.SLDASM/meshes/handgelenk.STL; visual mesh filename=package://RescueBot_Baugruppe.SLDASM/meshes/handgelenk.STL
- added link handgelenk2, mass 0.20444; collision mesh filename=package://RescueBot_Baugruppe.SLDASM/meshes/handgelenk2.STL; visual mesh filename=package://RescueBot_Baugruppe.SLDASM/meshes/handgelenk2.STL
- added link köchel, mass 0.038419; collision mesh filename=package://RescueBot_Baugruppe.SLDASM/meshes/köchel.STL; visual mesh filename=package://RescueBot_Baugruppe.SLDASM/meshes/köchel.STL
- added link schulterGelenk, mass 8.2963; collision mesh filename=package://RescueBot_Baugruppe.SLDASM/meshes/schulterGelenk.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; visual mesh filename=package://RescueBot_Baugruppe.SLDASM/meshes/schulterGelenk.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
- link base_link: mass 3.0727 -> 8.2963
Joints:
- removed joint Drehplatt
- removed joint Finger
- removed joint Hand
- removed joint Oberarm
- removed joint Unterarm
- added joint finger: type continuous, parent köchel, child fingergelenk, origin xyz=0.124825859230761 0 0 rpy=-3.14159265358979 0 3.14159265358979, axis 1 0 0
- added joint hand: type continuous, parent handgelenk, child handgelenk2, origin xyz=0 0 0.575 rpy=-1.96362785676128 0 0, axis 1 0 0
- added joint hand2: type continuous, parent handgelenk2, child köchel, origin xyz=0.00200000000000047 0 0.168317889650684 rpy=2.20889980848183 -1.5707963267949 0, axis 1 0 0
- added joint oberarm: type continuous, parent schulterGelenk, child ellenbogen, origin xyz=0 0.202999999999992 0.0249999999999935 rpy=-1.5707963267949 -0.740356965763116 1.5707963267949, axis 0 0 1
- added joint schulter: type fixed, parent base_link, child schulterGelenk, origin xyz=0 -0.799999999999999 0.448167457544184 rpy=1.5707963267949 0 2.86985130632957, axis 0 0 0
- added joint unterarm: type continuous, parent ellenbogen, child handgelenk, origin xyz=0.74500000000001 0 0 rpy=2.65796523927005 1.5707963267949 0, axis 1 0 0
